File: Master.kicad_sch (KiCad schematic)
At the start: 7 parts, among them J1 43045-1012

Commit message: Rename resistor R3 to R1 in Master sheet; refresh sheet UUIDs
Co-Authored-By: Claude Fable 5.1 <noreply@anthropic.com>
Parts:
- renumbered R3 to R1
Changed lines of the file:
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@@
 		(dnp no)
 		(fields_autoplaced yes)
-		(property "Reference" "R3"
+		(property "Reference" "R1"
 			(at 109.22 86.36 90)
 			(show_name no)
@@
 			(project "XDMX-WT"
 				(path "/81fc2a60-bc27-447a-859e-9589360cae3c/4fa36aa0-c61b-4d75-9356-c24a00001160"
-					(reference "R3")
+					(reference "R1")
 					(unit 1)
 				)
